File: Schaltplan.sch (EAGLE design)
At the start: 33 parts, among them IC1 74AHC1G04DBV, U1 TB6621FNG, U2 TB6621FNG, U3 TB6621FNG

Commit message: corrected Schaltplan
Parts:
- added R3: 1k, resistor:R-EU_0204/7
Changed lines of the file:
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@@
 <part name="IC3" library="v-reg" deviceset="LM323-TO3" device=""/>
 <part name="C10" library="capacitor-wima" deviceset="C" device="2,5-3"/>
-<part name="R2" library="docu-dummy" deviceset="R" device=""/>
+<part name="R2" library="docu-dummy" deviceset="R" device="" value="1k"/>
+<part name="R3" library="resistor" deviceset="R-EU_" device="0204/7" value="1k"/>
 </parts>
 <sheets>
@@
 <instance part="C10" gate="G$1" x="205.74" y="248.92"/>
 <instance part="R2" gate="G$1" x="129.54" y="309.88" rot="R180"/>
+<instance part="R3" gate="G$1" x="203.2" y="325.12"/>
 </instances>
 <busses>
@@
 <pinref part="C3" gate="G$1" pin="+"/>
 <pinref part="JP1" gate="G$1" pin="8"/>
-<wire x1="-185.42" y1="177.8" x2="-205.74" y2="177.8" width="0.1524" layer="91"/>
-<junction x="-185.42" y="177.8"/>
-<wire x1="-205.74" y1="177.8" x2="-205.74" y2="276.86" width="0.1524" layer="91"/>
 </segment>
 <segment>
@@
 <pinref part="C9" gate="G$1" pin="+"/>
 <pinref part="JP5" gate="G$1" pin="8"/>
-<wire x1="-182.88" y1="279.4" x2="-205.74" y2="279.4" width="0.1524" layer="91"/>
-<junction x="-182.88" y="279.4"/>
 </segment>
 </net>
@@
 <wire x1="-7.62" y1="187.96" x2="-17.78" y2="187.96" width="0.1524" layer="91"/>
 <junction x="-7.62" y="187.96"/>
+<junction x="-7.62" y="172.72"/>
 </segment>
 <segment>
@@
 <wire x1="137.16" y1="358.14" x2="137.16" y2="332.74" width="0.1524" layer="91"/>
 <junction x="66.04" y="358.14"/>
+<wire x1="66.04" y1="358.14" x2="-200.66" y2="358.14" width="0.1524" layer="91"/>
+<wire x1="-200.66" y1="358.14" x2="-200.66" y2="279.4" width="0.1524" layer="91"/>
+<wire x1="-200.66" y1="279.4" x2="-200.66" y2="177.8" width="0.1524" layer="91"/>
+<wire x1="-200.66" y1="177.8" x2="-185.42" y2="177.8" width="0.1524" layer="91"/>
+<wire x1="-200.66" y1="279.4" x2="-182.88" y2="279.4" width="0.1524" layer="91"/>
+<junction x="-200.66" y="279.4"/>
 </segment>
 </net>
@@
 </segment>
 </net>
+<net name="N$9" class="0">
+<segment>
+<wire x1="-205.74" y1="177.8" x2="-205.74" y2="276.86" width="0.1524" layer="91"/>
+</segment>
+</net>

Commit message: edited Schaltplan
Parts:
- added R2, R4: 1k, resistor:R-EU_0204/2V
- added R5: 2k, resistor:R-EU_0204/2V
- R3: value 1k -> 5 Ohm
- renumbered Q1 to BC237NPN
Connections:
- new net N$10: BC237NPN.B, R5.2
- net AIN2: now also R5.1
- net N$3: now also R2.2, R4.2
- net N$7: now also R4.1
- net N$8: now also R2.1
- net VCC: now also R3.1, R3.2
Other:
- note removed: "1k"
- moved on the sheet: R3
Changed lines of the file:
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@@
 <part name="P+6" library="SparkFun" deviceset="VCC" device="" value="RAW"/>
 <part name="IC1" library="74xx-little-de" deviceset="74*1G04" device="DBV" technology="AHC"/>
-<part name="R1" library="docu-dummy" deviceset="R" device=""/>
-<part name="Q1" library="semicon-smd-ipc" deviceset="NPN-TRANSISTIOR-2COL" device="SOT89"/>
+<part name="BC237NPN" library="semicon-smd-ipc" deviceset="NPN-TRANSISTIOR-2COL" device="SOT89"/>
 <part name="GND23" library="supply1" deviceset="GND" device=""/>
 <part name="GND24" library="supply1" deviceset="GND" device=""/>
@@
 <part name="IC3" library="v-reg" deviceset="LM323-TO3" device=""/>
 <part name="C10" library="capacitor-wima" deviceset="C" device="2,5-3"/>
-<part name="R2" library="docu-dummy" deviceset="R" device="" value="1k"/>
-<part name="R3" library="resistor" deviceset="R-EU_" device="0204/7" value="1k"/>
+<part name="R3" library="resistor" deviceset="R-EU_" device="0204/7" value="5 Ohm"/>
+<part name="R4" library="resistor" deviceset="R-EU_" device="0204/2V" value="1k"/>
+<part name="R2" library="resistor" deviceset="R-EU_" device="0204/2V" value="1k"/>
+<part name="R5" library="resistor" deviceset="R-EU_" device="0204/2V" value="2k"/>
 </parts>
 <sheets>
@@
 <text x="139.7" y="314.96" size="1.778" layer="91">12V</text>
 <text x="190.5" y="246.38" size="1.778" layer="91">0.1-10uF</text>
-<text x="127" y="304.8" size="1.778" layer="91">1k</text>
+<rectangle x1="-43.18" y1="180.34" x2="-12.7" y2="248.92" layer="91"/>
+<rectangle x1="269.24" y1="132.08" x2="284.48" y2="147.32" layer="91"/>
 </plain>
 <instances>
@@
 <instance part="P+6" gate="1" x="233.68" y="223.52"/>
 <instance part="IC1" gate="A" x="271.78" y="139.7"/>
-<instance part="R1" gate="G$1" x="320.04" y="33.02"/>
-<instance part="Q1" gate="G$1" x="327.66" y="33.02"/>
+<instance part="BC237NPN" gate="G$1" x="327.66" y="33.02"/>
 <instance part="GND23" gate="1" x="330.2" y="25.4"/>
 <instance part="GND24" gate="1" x="314.96" y="124.46"/>
@@
 <instance part="IC3" gate="G$1" x="137.16" y="325.12" rot="R270"/>
 <instance part="C10" gate="G$1" x="205.74" y="248.92"/>
-<instance part="R2" gate="G$1" x="129.54" y="309.88" rot="R180"/>
-<instance part="R3" gate="G$1" x="203.2" y="325.12"/>
+<instance part="R3" gate="G$1" x="444.5" y="71.12"/>
+<instance part="R4" gate="G$1" x="58.42" y="314.96" rot="R90"/>
+<instance part="R2" gate="G$1" x="129.54" y="314.96" rot="R90"/>
+<instance part="R5" gate="G$1" x="314.96" y="33.02"/>
 </instances>
 <busses>
@@
 </segment>
 <segment>
-<pinref part="Q1" gate="G$1" pin="E"/>
+<pinref part="BC237NPN" gate="G$1" pin="E"/>
 <pinref part="GND23" gate="1" pin="GND"/>
 </segment>
@@
 <wire x1="383.54" y1="71.12" x2="391.16" y2="71.12" width="0.1524" layer="91"/>
 <wire x1="391.16" y1="71.12" x2="398.78" y2="71.12" width="0.1524" layer="91"/>
-<wire x1="398.78" y1="71.12" x2="467.36" y2="71.12" width="0.1524" layer="91"/>
+<wire x1="398.78" y1="71.12" x2="439.42" y2="71.12" width="0.1524" layer="91"/>
+<wire x1="439.42" y1="71.12" x2="449.58" y2="71.12" width="0.1524" layer="91"/>
+<wire x1="449.58" y1="71.12" x2="467.36" y2="71.12" width="0.1524" layer="91"/>
 <wire x1="467.36" y1="71.12" x2="467.36" y2="109.22" width="0.1524" layer="91"/>
 <junction x="467.36" y="109.22"/>
@@
 <pinref part="LED9" gate="G$1" pin="A"/>
 <junction x="398.78" y="71.12"/>
+<pinref part="R3" gate="G$1" pin="2"/>
+<junction x="449.58" y="71.12"/>
+<pinref part="R3" gate="G$1" pin="1"/>
+<junction x="439.42" y="71.12"/>
 </segment>
 <segment>
@@
 <wire x1="266.7" y1="99.06" x2="226.06" y2="99.06" width="0.1524" layer="91"/>
 <junction x="266.7" y="99.06"/>
-<wire x1="314.96" y1="33.02" x2="266.7" y2="33.02" width="0.1524" layer="91"/>
+<wire x1="314.96" y1="33.02" x2="309.88" y2="33.02" width="0.1524" layer="91"/>
+<pinref part="R5" gate="G$1" pin="1"/>
+<wire x1="309.88" y1="33.02" x2="266.7" y2="33.02" width="0.1524" layer="91"/>
+<junction x="309.88" y="33.02"/>
 </segment>
 <segment>
@@
 <segment>
 <pinref part="LED12" gate="G$1" pin="C"/>
-<pinref part="Q1" gate="G$1" pin="C/"/>
+<pinref part="BC237NPN" gate="G$1" pin="C/"/>
 <wire x1="398.78" y1="55.88" x2="330.2" y2="55.88" width="0.1524" layer="91"/>
 <wire x1="330.2" y1="55.88" x2="330.2" y2="35.56" width="0.1524" layer="91"/>
@@
 <wire x1="205.74" y1="251.46" x2="205.74" y2="256.54" width="0.1524" layer="91"/>
 <junction x="205.74" y="256.54"/>
-<wire x1="124.46" y1="309.88" x2="124.46" y2="325.12" width="0.1524" layer="91"/>
-<wire x1="124.46" y1="325.12" x2="129.54" y2="325.12" width="0.1524" layer="91"/>
+<pinref part="R4" gate="G$1" pin="2"/>
+<wire x1="58.42" y1="325.12" x2="58.42" y2="320.04" width="0.1524" layer="91"/>
+<junction x="58.42" y="325.12"/>
+<pinref part="R2" gate="G$1" pin="2"/>
+<wire x1="129.54" y1="320.04" x2="129.54" y2="325.12" width="0.1524" layer="91"/>
 <junction x="129.54" y="325.12"/>
 </segment>
@@
 <segment>
 <pinref part="IC2" gate="G$1" pin="OUT"/>
-<wire x1="66.04" y1="317.5" x2="66.04" y2="279.4" width="0.1524" layer="91"/>
+<wire x1="66.04" y1="317.5" x2="66.04" y2="309.88" width="0.1524" layer="91"/>
+<wire x1="66.04" y1="309.88" x2="66.04" y2="279.4" width="0.1524" layer="91"/>
 <wire x1="104.14" y1="279.4" x2="480.06" y2="279.4" width="0.1524" layer="91"/>
 <wire x1="480.06" y1="279.4" x2="480.06" y2="172.72" width="0.1524" layer="91"/>
@@
 <wire x1="205.74" y1="243.84" x2="205.74" y2="238.76" width="0.1524" layer="91"/>
 <junction x="205.74" y="238.76"/>
+<pinref part="R4" gate="G$1" pin="1"/>
+<wire x1="58.42" y1="309.88" x2="66.04" y2="309.88" width="0.1524" layer="91"/>
+<junction x="66.04" y="309.88"/>
 </segment>
 </net>
@@
 <wire x1="134.62" y1="309.88" x2="137.16" y2="309.88" width="0.1524" layer="91"/>
 <junction x="137.16" y="309.88"/>
+<pinref part="R2" gate="G$1" pin="1"/>
+<wire x1="129.54" y1="309.88" x2="137.16" y2="309.88" width="0.1524" layer="91"/>
 </segment>
 </net>
@@
 </segment>
 </net>
+<net name="N$10" class="0">
+<segment>
+<pinref part="BC237NPN" gate="G$1" pin="B"/>
+<wire x1="317.5" y1="33.02" x2="320.04" y2="33.02" width="0.1524" layer="91"/>
+<pinref part="R5" gate="G$1" pin="2"/>
+<wire x1="320.04" y1="33.02" x2="325.12" y2="33.02" width="0.1524" layer="91"/>
+<junction x="320.04" y="33.02"/>
+</segment>
+</net>

Commit message: edited Schaltplan
Parts:
- removed LED7, LED8, LED9: (no value), led:LED
- removed R3: 5 Ohm, resistor:R-EU_0204/7
- added R1, R6, R7: 51 Ohm, resistor:R-EU_0204/2V
- R2, R4: value 1k -> 10k
Connections:
- removed net N$1: BC237NPN.C/, LED12.C
- new net N$11: BC237NPN.C, LED10.C, LED11.C, LED12.C
- net N$4: now also R1.1; no longer LED7.C
- net N$5: now also R6.1; no longer LED8.C
- net N$6: now also R7.1; no longer LED9.C
- net VCC: now also R1.2, R6.2, R7.2; no longer LED7.A, LED8.A, LED9.A, R3.1, R3.2
Other:
- moved on the sheet: BC237NPN, LED10, LED11, LED12, R5
Changed lines of the file:
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@@
 <part name="GND23" library="supply1" deviceset="GND" device=""/>
 <part name="GND24" library="supply1" deviceset="GND" device=""/>
-<part name="LED7" library="led" deviceset="LED" device=""/>
-<part name="LED8" library="led" deviceset="LED" device=""/>
-<part name="LED9" library="led" deviceset="LED" device=""/>
 <part name="LED10" library="led" deviceset="LED" device=""/>
 <part name="LED11" library="led" deviceset="LED" device=""/>
@@
 <part name="IC3" library="v-reg" deviceset="LM323-TO3" device=""/>
 <part name="C10" library="capacitor-wima" deviceset="C" device="2,5-3"/>
-<part name="R3" library="resistor" deviceset="R-EU_" device="0204/7" value="5 Ohm"/>
-<part name="R4" library="resistor" deviceset="R-EU_" device="0204/2V" value="1k"/>
-<part name="R2" library="resistor" deviceset="R-EU_" device="0204/2V" value="1k"/>
+<part name="R4" library="resistor" deviceset="R-EU_" device="0204/2V" value="10k"/>
+<part name="R2" library="resistor" deviceset="R-EU_" device="0204/2V" value="10k"/>
 <part name="R5" library="resistor" deviceset="R-EU_" device="0204/2V" value="2k"/>
+<part name="R1" library="resistor" deviceset="R-EU_" device="0204/2V" value="51 Ohm"/>
+<part name="R6" library="resistor" deviceset="R-EU_" device="0204/2V" value="51 Ohm"/>
+<part name="R7" library="resistor" deviceset="R-EU_" device="0204/2V" value="51 Ohm"/>
 </parts>
 <sheets>
@@
 <text x="139.7" y="314.96" size="1.778" layer="91">12V</text>
 <text x="190.5" y="246.38" size="1.778" layer="91">0.1-10uF</text>
-<rectangle x1="-43.18" y1="180.34" x2="-12.7" y2="248.92" layer="91"/>
-<rectangle x1="269.24" y1="132.08" x2="284.48" y2="147.32" layer="91"/>
 </plain>
 <instances>
@@
 <instance part="P+6" gate="1" x="233.68" y="223.52"/>
 <instance part="IC1" gate="A" x="271.78" y="139.7"/>
-<instance part="BC237NPN" gate="G$1" x="327.66" y="33.02"/>
-<instance part="GND23" gate="1" x="330.2" y="25.4"/>
+<instance part="BC237NPN" gate="G$1" x="462.28" y="33.02"/>
+<instance part="GND23" gate="1" x="464.82" y="25.4"/>
 <instance part="GND24" gate="1" x="314.96" y="124.46"/>
-<instance part="LED7" gate="G$1" x="383.54" y="68.58"/>
-<instance part="LED8" gate="G$1" x="391.16" y="68.58"/>
-<instance part="LED9" gate="G$1" x="398.78" y="68.58"/>
-<instance part="LED10" gate="G$1" x="383.54" y="60.96"/>
-<instance part="LED11" gate="G$1" x="391.16" y="60.96"/>
-<instance part="LED12" gate="G$1" x="398.78" y="60.96"/>
+<instance part="LED10" gate="G$1" x="459.74" y="66.04"/>
+<instance part="LED11" gate="G$1" x="467.36" y="66.04"/>
+<instance part="LED12" gate="G$1" x="474.98" y="66.04"/>
 <instance part="IC2" gate="G$1" x="66.04" y="325.12" rot="R270"/>
 <instance part="IC3" gate="G$1" x="137.16" y="325.12" rot="R270"/>
 <instance part="C10" gate="G$1" x="205.74" y="248.92"/>
-<instance part="R3" gate="G$1" x="444.5" y="71.12"/>
 <instance part="R4" gate="G$1" x="58.42" y="314.96" rot="R90"/>
 <instance part="R2" gate="G$1" x="129.54" y="314.96" rot="R90"/>
-<instance part="R5" gate="G$1" x="314.96" y="33.02"/>
+<instance part="R5" gate="G$1" x="449.58" y="33.02"/>
+<instance part="R1" gate="G$1" x="459.74" y="76.2" rot="R90"/>
+<instance part="R6" gate="G$1" x="467.36" y="76.2" rot="R90"/>
+<instance part="R7" gate="G$1" x="474.98" y="76.2" rot="R90"/>
 </instances>
 <busses>
@@
 <junction x="467.36" y="142.24"/>
 <wire x1="480.06" y1="142.24" x2="480.06" y2="172.72" width="0.1524" layer="91"/>
-<wire x1="383.54" y1="71.12" x2="391.16" y2="71.12" width="0.1524" layer="91"/>
-<wire x1="391.16" y1="71.12" x2="398.78" y2="71.12" width="0.1524" layer="91"/>
-<wire x1="398.78" y1="71.12" x2="439.42" y2="71.12" width="0.1524" layer="91"/>
-<wire x1="439.42" y1="71.12" x2="449.58" y2="71.12" width="0.1524" layer="91"/>
-<wire x1="449.58" y1="71.12" x2="467.36" y2="71.12" width="0.1524" layer="91"/>
-<wire x1="467.36" y1="71.12" x2="467.36" y2="109.22" width="0.1524" layer="91"/>
 <junction x="467.36" y="109.22"/>
-<pinref part="LED7" gate="G$1" pin="A"/>
-<pinref part="LED8" gate="G$1" pin="A"/>
-<junction x="391.16" y="71.12"/>
-<pinref part="LED9" gate="G$1" pin="A"/>
-<junction x="398.78" y="71.12"/>
-<pinref part="R3" gate="G$1" pin="2"/>
-<junction x="449.58" y="71.12"/>
-<pinref part="R3" gate="G$1" pin="1"/>
-<junction x="439.42" y="71.12"/>
+<pinref part="R1" gate="G$1" pin="2"/>
+<wire x1="467.36" y1="81.28" x2="467.36" y2="109.22" width="0.1524" layer="91"/>
+<wire x1="459.74" y1="81.28" x2="467.36" y2="81.28" width="0.1524" layer="91"/>
+<pinref part="R6" gate="G$1" pin="2"/>
+<junction x="467.36" y="81.28"/>
+<pinref part="R7" gate="G$1" pin="2"/>
+<wire x1="474.98" y1="81.28" x2="467.36" y2="81.28" width="0.1524" layer="91"/>
 </segment>
 <segment>
@@
 <wire x1="266.7" y1="99.06" x2="226.06" y2="99.06" width="0.1524" layer="91"/>
 <junction x="266.7" y="99.06"/>
-<wire x1="314.96" y1="33.02" x2="309.88" y2="33.02" width="0.1524" layer="91"/>
+<wire x1="449.58" y1="33.02" x2="444.5" y2="33.02" width="0.1524" layer="91"/>
 <pinref part="R5" gate="G$1" pin="1"/>
-<wire x1="309.88" y1="33.02" x2="266.7" y2="33.02" width="0.1524" layer="91"/>
-<junction x="309.88" y="33.02"/>
+<wire x1="444.5" y1="33.02" x2="266.7" y2="33.02" width="0.1524" layer="91"/>
+<junction x="444.5" y="33.02"/>
 </segment>
 <segment>
@@
 </segment>
 </net>
-<net name="N$4" class="0">
-<segment>
-<pinref part="LED7" gate="G$1" pin="C"/>
-<pinref part="LED10" gate="G$1" pin="A"/>
-</segment>
-</net>
-<net name="N$5" class="0">
-<segment>
-<pinref part="LED8" gate="G$1" pin="C"/>
-<pinref part="LED11" gate="G$1" pin="A"/>
-</segment>
-</net>
-<net name="N$6" class="0">
-<segment>
-<pinref part="LED9" gate="G$1" pin="C"/>
-<pinref part="LED12" gate="G$1" pin="A"/>
-</segment>
-</net>
-<net name="N$1" class="0">
-<segment>
-<pinref part="LED12" gate="G$1" pin="C"/>
-<pinref part="BC237NPN" gate="G$1" pin="C/"/>
-<wire x1="398.78" y1="55.88" x2="330.2" y2="55.88" width="0.1524" layer="91"/>
-<wire x1="330.2" y1="55.88" x2="330.2" y2="35.56" width="0.1524" layer="91"/>
-</segment>
-</net>
 <net name="N$2" class="0">
 <segment>
@@
 <wire x1="129.54" y1="320.04" x2="129.54" y2="325.12" width="0.1524" layer="91"/>
 <junction x="129.54" y="325.12"/>
+<wire x1="116.84" y1="256.54" x2="116.84" y2="180.34" width="0.1524" layer="91"/>
+<junction x="116.84" y="256.54"/>
+<wire x1="116.84" y1="180.34" x2="78.74" y2="180.34" width="0.1524" layer="91"/>
 </segment>
 </net>
@@
 <segment>
 <pinref part="BC237NPN" gate="G$1" pin="B"/>
-<wire x1="317.5" y1="33.02" x2="320.04" y2="33.02" width="0.1524" layer="91"/>
+<wire x1="452.12" y1="33.02" x2="454.66" y2="33.02" width="0.1524" layer="91"/>
 <pinref part="R5" gate="G$1" pin="2"/>
-<wire x1="320.04" y1="33.02" x2="325.12" y2="33.02" width="0.1524" layer="91"/>
-<junction x="320.04" y="33.02"/>
-</segment>
-</net>
+<wire x1="454.66" y1="33.02" x2="459.74" y2="33.02" width="0.1524" layer="91"/>
+<junction x="454.66" y="33.02"/>
+</segment>
+</net>
+<net name="N$4" class="0">
+<segment>
+<pinref part="R1" gate="G$1" pin="1"/>
+<pinref part="LED10" gate="G$1" pin="A"/>
+<wire x1="459.74" y1="71.12" x2="459.74" y2="68.58" width="0.1524" layer="91"/>
+</segment>
+</net>
+<net name="N$5" class="0">
+<segment>
+<pinref part="R6" gate="G$1" pin="1"/>
+<pinref part="LED11" gate="G$1" pin="A"/>
+<wire x1="467.36" y1="71.12" x2="467.36" y2="68.58" width="0.1524" layer="91"/>
+</segment>
+</net>
+<net name="N$6" class="0">
+<segment>
+<pinref part="R7" gate="G$1" pin="1"/>
+<pinref part="LED12" gate="G$1" pin="A"/>
+<wire x1="474.98" y1="71.12" x2="474.98" y2="68.58" width="0.1524" layer="91"/>
+</segment>
+</net>
+<net name="N$11" class="0">
+<segment>
+<pinref part="LED12" gate="G$1" pin="C"/>
+<wire x1="474.98" y1="60.96" x2="467.36" y2="60.96" width="0.1524" layer="91"/>
+<pinref part="LED11" gate="G$1" pin="C"/>
+<junction x="467.36" y="60.96"/>
+<wire x1="467.36" y1="60.96" x2="459.74" y2="60.96" width="0.1524" layer="91"/>
+<pinref part="LED10" gate="G$1" pin="C"/>
+<pinref part="BC237NPN" gate="G$1" pin="C"/>
+<wire x1="467.36" y1="60.96" x2="464.82" y2="60.96" width="0.1524" layer="91"/>
+<wire x1="464.82" y1="60.96" x2="464.82" y2="38.1" width="0.1524" layer="91"/>
+</segment>
+</net>
